Commit message: update lerobot_0.4.4 branch support and adapt the current gripper setup in the URDF

File: mani_skill/assets/robots/so100/so100.urdf (robot description, URDF)
Before this commit: robot SO_5DOF_ARM100_8j_URDF.SLDASM, 9 links, 8 joints
Joints:
- joint gripper: limit lower=-1.1 upper=1.1 effort=0 velocity=0 -> lower=-0.876 upper=0.876 effort=0 velocity=0; origin xyz=-0.0202 -0.0244 0 rpy=0 3.14159 -0.9 -> xyz=-0.0202 -0.0244 0 rpy=0 3.14159 -0.695
- joint wrist_flex: axis 1 0 0 -> -1 0 0; origin xyz=0 0.0052 0.1349 rpy=-1.5708 0 0 -> xyz=0 0.0052 0.1349 rpy=-1.5708 0 3.14
- joint wrist_roll: origin xyz=0 -0.0601 0 rpy=0 1.5708 0 -> xyz=0 -0.0601 0 rpy=0 -1.5708 0
